File: staypuft.sch (KiCad schematic (older format))
At the start: 55 parts, among them Q1 2N5088, Q2 2N5088, Q3 2N5088, Q4 2N5088

Commit message: updated values
Parts:
- C1: value CP -> 20u
- C10, C3, C7: value C -> 470p
- C11: value C -> 3.9n
- C12: value C -> 10n
- C13, C14, C2, C4, C5, C8: value C -> 100n
- C6, C9: value C -> 47n
- R1: value R -> 39k
- R10, R15, R4: value R -> 12k
- R11, R16, R5: value R -> 390
- R12, R21, R7: value R -> 10k
- R13, R2, R20, R9: value R -> 100k
- R14, R19, R3, R8: value R -> 470k
- R17: value R -> 20k
- R18: value R -> 22k
- R22: value R -> 2.7k
- R6: value R -> 1k
- RV1, RV2, RV3: value R_POT -> 100k
Changed lines of the file:
@@
 encoding utf-8
 Sheet 1 1
-Title ""
-Date ""
-Rev ""
-Comp ""
-Comment1 ""
+Title "Stay Puft Fuzz"
+Date "2021-05-01"
+Rev "v1.0"
+Comp ":P"
+Comment1 "Two possible FB mods are here"
 Comment2 ""
 Comment3 ""
@@
 P 1450 3900
 F 0 "R1" V 1243 3900 50  0000 C CNN
-F 1 "R" V 1334 3900 50  0000 C CNN
+F 1 "39k" V 1334 3900 50  0000 C CNN
 F 2 "" V 1380 3900 50  0001 C CNN
 F 3 "~" H 1450 3900 50  0001 C CNN
@@
 P 2550 3600
 F 0 "R3" V 2343 3600 50  0000 C CNN
-F 1 "R" V 2434 3600 50  0000 C CNN
+F 1 "470k" V 2434 3600 50  0000 C CNN
 F 2 "" V 2480 3600 50  0001 C CNN
 F 3 "~" H 2550 3600 50  0001 C CNN
@@
 P 2100 4450
 F 0 "R2" H 2030 4404 50  0000 R CNN
-F 1 "R" H 2030 4495 50  0000 R CNN
+F 1 "100k" H 2030 4495 50  0000 R CNN
 F 2 "" V 2030 4450 50  0001 C CNN
 F 3 "~" H 2100 4450 50  0001 C CNN
@@
 P 3050 4450
 F 0 "R5" H 2980 4404 50  0000 R CNN
-F 1 "R" H 2980 4495 50  0000 R CNN
+F 1 "390" H 2980 4495 50  0000 R CNN
 F 2 "" V 2980 4450 50  0001 C CNN
 F 3 "~" H 3050 4450 50  0001 C CNN
@@
 P 3650 4450
 F 0 "R6" H 3580 4404 50  0000 R CNN
-F 1 "R" H 3580 4495 50  0000 R CNN
+F 1 "1k" H 3580 4495 50  0000 R CNN
 F 2 "" V 3580 4450 50  0001 C CNN
 F 3 "~" H 3650 4450 50  0001 C CNN
@@
 P 3050 2400
 F 0 "R4" H 2980 2354 50  0000 R CNN
-F 1 "R" H 2980 2445 50  0000 R CNN
+F 1 "12k" H 2980 2445 50  0000 R CNN
 F 2 "" V 2980 2400 50  0001 C CNN
 F 3 "~" H 3050 2400 50  0001 C CNN
@@
 P 4300 3900
 F 0 "R7" V 4507 3900 50  0000 C CNN
-F 1 "R" V 4416 3900 50  0000 C CNN
+F 1 "10k" V 4416 3900 50  0000 C CNN
 F 2 "" V 4230 3900 50  0001 C CNN
 F 3 "~" H 4300 3900 50  0001 C CNN
@@
 U 1 1 608EB3F0
 P 5000 3600
-F 0 "R8" V 4793 3600 50  0000 C CNN
-F 1 "R" V 4884 3600 50  0000 C CNN
+F 0 "R8" V 4950 3750 50  0000 C CNN
+F 1 "470k" V 5100 3600 50  0000 C CNN
 F 2 "" V 4930 3600 50  0001 C CNN
 F 3 "~" H 5000 3600 50  0001 C CNN
@@
 P 5000 4450
 F 0 "R9" H 4930 4404 50  0000 R CNN
-F 1 "R" H 4930 4495 50  0000 R CNN
+F 1 "100k" H 4930 4495 50  0000 R CNN
 F 2 "" V 4930 4450 50  0001 C CNN
 F 3 "~" H 5000 4450 50  0001 C CNN
@@
 P 5400 4450
 F 0 "R11" H 5330 4404 50  0000 R CNN
-F 1 "R" H 5330 4495 50  0000 R CNN
+F 1 "390" H 5330 4495 50  0000 R CNN
 F 2 "" V 5330 4450 50  0001 C CNN
 F 3 "~" H 5400 4450 50  0001 C CNN
@@
 P 5400 2400
 F 0 "R10" H 5330 2354 50  0000 R CNN
-F 1 "R" H 5330 2445 50  0000 R CNN
+F 1 "12k" H 5330 2445 50  0000 R CNN
 F 2 "" V 5330 2400 50  0001 C CNN
 F 3 "~" H 5400 2400 50  0001 C CNN
@@
 P 6250 3900
 F 0 "R12" V 6457 3900 50  0000 C CNN
-F 1 "R" V 6366 3900 50  0000 C CNN
+F 1 "10k" V 6366 3900 50  0000 C CNN
 F 2 "" V 6180 3900 50  0001 C CNN
 F 3 "~" H 6250 3900 50  0001 C CNN
@@
 P 7450 4450
 F 0 "R16" H 7520 4496 50  0000 L CNN
-F 1 "R" H 7520 4405 50  0000 L CNN
+F 1 "390" H 7520 4405 50  0000 L CNN
 F 2 "" V 7380 4450 50  0001 C CNN
 F 3 "~" H 7450 4450 50  0001 C CNN
@@
 P 6900 4450
 F 0 "R13" H 6970 4496 50  0000 L CNN
-F 1 "R" H 6970 4405 50  0000 L CNN
+F 1 "100k" H 6970 4405 50  0000 L CNN
 F 2 "" V 6830 4450 50  0001 C CNN
 F 3 "~" H 6900 4450 50  0001 C CNN
@@
 P 1850 3900
 F 0 "C2" V 1598 3900 50  0000 C CNN
-F 1 "C" V 1689 3900 50  0000 C CNN
+F 1 "100n" V 1689 3900 50  0000 C CNN
 F 2 "" H 1888 3750 50  0001 C CNN
 F 3 "~" H 1850 3900 50  0001 C CNN
@@
 P 3350 2700
 F 0 "C4" V 3098 2700 50  0000 C CNN
-F 1 "C" V 3189 2700 50  0000 C CNN
+F 1 "100n" V 3189 2700 50  0000 C CNN
 F 2 "" H 3388 2550 50  0001 C CNN
 F 3 "~" H 3350 2700 50  0001 C CNN
@@
 P 2550 2700
 F 0 "C3" V 2298 2700 50  0000 C CNN
-F 1 "C" V 2389 2700 50  0000 C CNN
+F 1 "470p" V 2389 2700 50  0000 C CNN
 F 2 "" H 2588 2550 50  0001 C CNN
 F 3 "~" H 2550 2700 50  0001 C CNN
@@
 P 4000 3900
 F 0 "C5" V 3748 3900 50  0000 C CNN
-F 1 "C" V 3839 3900 50  0000 C CNN
+F 1 "100n" V 3839 3900 50  0000 C CNN
 F 2 "" H 4038 3750 50  0001 C CNN
 F 3 "~" H 4000 3900 50  0001 C CNN
@@
 U 1 1 608F292A
 P 5000 3350
-F 0 "C7" V 4748 3350 50  0000 C CNN
-F 1 "C" V 4839 3350 50  0000 C CNN
+F 0 "C7" V 4950 3500 50  0000 C CNN
+F 1 "470p" V 4839 3350 50  0000 C CNN
 F 2 "" H 5038 3200 50  0001 C CNN
 F 3 "~" H 5000 3350 50  0001 C CNN
@@
 P 4700 2700
 F 0 "C6" V 4448 2700 50  0000 C CNN
-F 1 "C" V 4539 2700 50  0000 C CNN
+F 1 "47n" V 4539 2700 50  0000 C CNN
 F 2 "" H 4738 2550 50  0001 C CNN
 F 3 "~" H 4700 2700 50  0001 C CNN
@@
 P 3650 3900
 F 0 "RV1" H 3581 3946 50  0000 R CNN
-F 1 "R_POT" H 3581 3855 50  0000 R CNN
+F 1 "100k" H 3581 3855 50  0000 R CNN
 F 2 "" H 3650 3900 50  0001 C CNN
 F 3 "~" H 3650 3900 50  0001 C CNN
@@
 U 1 1 60968A94
 P 7050 3600
-F 0 "R14" V 6843 3600 50  0000 C CNN
-F 1 "R" V 6934 3600 50  0000 C CNN
+F 0 "R14" V 7000 3800 50  0000 C CNN
+F 1 "470k" V 7150 3600 50  0000 C CNN
 F 2 "" V 6980 3600 50  0001 C CNN
 F 3 "~" H 7050 3600 50  0001 C CNN
@@
 P 7450 2400
 F 0 "R15" H 7380 2354 50  0000 R CNN
-F 1 "R" H 7380 2445 50  0000 R CNN
+F 1 "12k" H 7380 2445 50  0000 R CNN
 F 2 "" V 7380 2400 50  0001 C CNN
 F 3 "~" H 7450 2400 50  0001 C CNN
@@
 U 1 1 60968AA8
 P 7050 3350
-F 0 "C10" V 6798 3350 50  0000 C CNN
-F 1 "C" V 6889 3350 50  0000 C CNN
+F 0 "C10" V 7000 3500 50  0000 C CNN
+F 1 "470p" V 6889 3350 50  0000 C CNN
 F 2 "" H 7088 3200 50  0001 C CNN
 F 3 "~" H 7050 3350 50  0001 C CNN
@@
 P 6750 2700
 F 0 "C9" V 6498 2700 50  0000 C CNN
-F 1 "C" V 6589 2700 50  0000 C CNN
+F 1 "47n" V 6589 2700 50  0000 C CNN
 F 2 "" H 6788 2550 50  0001 C CNN
 F 3 "~" H 6750 2700 50  0001 C CNN
@@
 P 5900 3900
 F 0 "C8" V 5648 3900 50  0000 C CNN
-F 1 "C" V 5739 3900 50  0000 C CNN
+F 1 "100n" V 5739 3900 50  0000 C CNN
 F 2 "" H 5938 3750 50  0001 C CNN
 F 3 "~" H 5900 3900 50  0001 C CNN
@@
 P 8350 3900
 F 0 "RV2" H 8281 3946 50  0000 R CNN
-F 1 "R_POT" H 8281 3855 50  0000 R CNN
+F 1 "100k" H 8281 3855 50  0000 R CNN
 F 2 "" H 8350 3900 50  0001 C CNN
 F 3 "~" H 8350 3900 50  0001 C CNN
@@
 P 7950 3600
 F 0 "C11" V 7698 3600 50  0000 C CNN
-F 1 "C" V 7789 3600 50  0000 C CNN
+F 1 "3.9n" V 7789 3600 50  0000 C CNN
 F 2 "" H 7988 3450 50  0001 C CNN
 F 3 "~" H 7950 3600 50  0001 C CNN
@@
 P 8700 3900
 F 0 "C13" V 8448 3900 50  0000 C CNN
-F 1 "C" V 8539 3900 50  0000 C CNN
+F 1 "100n" V 8539 3900 50  0000 C CNN
 F 2 "" H 8738 3750 50  0001 C CNN
 F 3 "~" H 8700 3900 50  0001 C CNN
@@
 P 8350 4450
 F 0 "C12" H 8235 4404 50  0000 R CNN
-F 1 "C" H 8235 4495 50  0000 R CNN
+F 1 "10n" H 8235 4495 50  0000 R CNN
 F 2 "" H 8388 4300 50  0001 C CNN
 F 3 "~" H 8350 4450 50  0001 C CNN
@@
 P 9850 3600
 F 0 "C14" V 9598 3600 50  0000 C CNN
-F 1 "C" V 9689 3600 50  0000 C CNN
+F 1 "100n" V 9689 3600 50  0000 C CNN
 F 2 "" H 9888 3450 50  0001 C CNN
 F 3 "~" H 9850 3600 50  0001 C CNN
@@
 P 7950 4150
 F 0 "R17" V 7743 4150 50  0000 C CNN
-F 1 "R" V 7834 4150 50  0000 C CNN
+F 1 "20k" V 7834 4150 50  0000 C CNN
 F 2 "" V 7880 4150 50  0001 C CNN
 F 3 "~" H 7950 4150 50  0001 C CNN
@@
 P 8350 3000
 F 0 "R18" H 8280 2954 50  0000 R CNN
-F 1 "R" H 8280 3045 50  0000 R CNN
+F 1 "22k" H 8280 3045 50  0000 R CNN
 F 2 "" V 8280 3000 50  0001 C CNN
 F 3 "~" H 8350 3000 50  0001 C CNN
@@
 P 9050 4450
 F 0 "R20" H 8980 4404 50  0000 R CNN
-F 1 "R" H 8980 4495 50  0000 R CNN
+F 1 "100k" H 8980 4495 50  0000 R CNN
 F 2 "" V 8980 4450 50  0001 C CNN
 F 3 "~" H 9050 4450 50  0001 C CNN
@@
 P 9050 2400
 F 0 "R19" H 8980 2354 50  0000 R CNN
-F 1 "R" H 8980 2445 50  0000 R CNN
+F 1 "470k" H 8980 2445 50  0000 R CNN
 F 2 "" V 8980 2400 50  0001 C CNN
 F 3 "~" H 9050 2400 50  0001 C CNN
@@
 P 9450 2400
 F 0 "R21" H 9380 2354 50  0000 R CNN
-F 1 "R" H 9380 2445 50  0000 R CNN
+F 1 "10k" H 9380 2445 50  0000 R CNN
 F 2 "" V 9380 2400 50  0001 C CNN
 F 3 "~" H 9450 2400 50  0001 C CNN
@@
 P 9450 4450
 F 0 "R22" H 9380 4404 50  0000 R CNN
-F 1 "R" H 9380 4495 50  0000 R CNN
+F 1 "2.7k" H 9380 4495 50  0000 R CNN
 F 2 "" V 9380 4450 50  0001 C CNN
 F 3 "~" H 9450 4450 50  0001 C CNN
@@
 P 10250 3900
 F 0 "RV3" H 10181 3946 50  0000 R CNN
-F 1 "R_POT" H 10181 3855 50  0000 R CNN
+F 1 "100k" H 10181 3855 50  0000 R CNN
 F 2 "" H 10250 3900 50  0001 C CNN
 F 3 "~" H 10250 3900 50  0001 C CNN
@@
 P 1500 2250
 F 0 "C1" H 1618 2296 50  0000 L CNN
-F 1 "CP" H 1618 2205 50  0000 L CNN
+F 1 "20u" H 1618 2205 50  0000 L CNN
 F 2 "" H 1538 2100 50  0001 C CNN
 F 3 "~" H 1500 2250 50  0001 C CNN

Commit message: choosing footprints
Parts:
- removed TP1, TP2: TestPoint, symbol Connector:TestPoint
- removed TP3: IN, symbol Connector:TestPoint
- removed TP8: OUT, symbol Connector:TestPoint
- added J1: Conn_01x04_Male, Connector_PinSocket_2.54mm:PinSocket_1x04_P2.54mm_Vertical, symbol Connector:Conn_01x04_Male
- D1, D2, D3, D4: footprint (none) -> Diode_THT:D_DO-35_SOD27_P10.16mm_Horizontal
- Q1, Q2, Q3, Q4: footprint Package_TO_SOT_THT:TO-92_Inline -> Package_TO_SOT_THT:TO-92_Inline_Wide
- R1, R10, R11, R12, R13, R14, R15, R16, R17, R18, R19, R2, R20, R21, R22, R3, R4, R5, R6, R7, R8, R9: footprint (none) -> Resistor_THT:R_Axial_DIN0207_L6.3mm_D2.5mm_P10.16mm_Horizontal
- RV3: footprint (none) -> Potentiometer_THT:Potentiometer_Omeg_PC16BU_Vertical
- TP4, TP5, TP6, TP7: footprint (none) -> Connector_PinHeader_2.54mm:PinHeader_1x01_P2.54mm_Vertical
Connections:
- net +9V: now also J1.1 (Pin_1)
- net GND: now also J1.4 (Pin_4)
- net in: now reaches R1.2
- net in: now also J1.2 (Pin_2)
- net out: now reaches RV3.2
- net out: now also J1.3 (Pin_3)

Commit message: finished footprint association
Parts:
- added D5: 1n4001, Diode_THT:D_DO-41_SOD81_P10.16mm_Horizontal, symbol Device:D
- C1: footprint (none) -> Capacitor_THT:CP_Radial_D5.0mm_P2.50mm
- C10, C3, C7: footprint (none) -> Capacitor_THT:C_Disc_D5.0mm_W2.5mm_P5.00mm
- C11, C12, C13, C14, C2, C4, C5, C6, C8, C9: footprint (none) -> Capacitor_THT:C_Rect_L7.2mm_W3.0mm_P5.00mm_FKS2_FKP2_MKS2_MKP2
- RV1, RV2: footprint (none) -> TerminalBlock:TerminalBlock_bornier-3_P5.08mm
Connections:
- net +9V: now also D5.1 (K)
- net GND: now also D5.2 (A)
Other:
- moved on the sheet: C1
Changed lines of the file:
@@
 F 0 "C2" V 1598 3900 50  0000 C CNN
 F 1 "100n" V 1689 3900 50  0000 C CNN
-F 2 "" H 1888 3750 50  0001 C CNN
+F 2 "Capacitor_THT:C_Rect_L7.2mm_W3.0mm_P5.00mm_FKS2_FKP2_MKS2_MKP2" H 1888 3750 50  0001 C CNN
 F 3 "~" H 1850 3900 50  0001 C CNN
 	1    1850 3900
@@
 F 0 "C4" V 3098 2700 50  0000 C CNN
 F 1 "100n" V 3189 2700 50  0000 C CNN
-F 2 "" H 3388 2550 50  0001 C CNN
+F 2 "Capacitor_THT:C_Rect_L7.2mm_W3.0mm_P5.00mm_FKS2_FKP2_MKS2_MKP2" H 3388 2550 50  0001 C CNN
 F 3 "~" H 3350 2700 50  0001 C CNN
 	1    3350 2700
@@
 F 0 "C3" V 2298 2700 50  0000 C CNN
 F 1 "470p" V 2389 2700 50  0000 C CNN
-F 2 "" H 2588 2550 50  0001 C CNN
+F 2 "Capacitor_THT:C_Disc_D5.0mm_W2.5mm_P5.00mm" H 2588 2550 50  0001 C CNN
 F 3 "~" H 2550 2700 50  0001 C CNN
 	1    2550 2700
@@
 F 0 "C5" V 3748 3900 50  0000 C CNN
 F 1 "100n" V 3839 3900 50  0000 C CNN
-F 2 "" H 4038 3750 50  0001 C CNN
+F 2 "Capacitor_THT:C_Rect_L7.2mm_W3.0mm_P5.00mm_FKS2_FKP2_MKS2_MKP2" H 4038 3750 50  0001 C CNN
 F 3 "~" H 4000 3900 50  0001 C CNN
 	1    4000 3900
@@
 F 0 "C7" V 4950 3500 50  0000 C CNN
 F 1 "470p" V 4839 3350 50  0000 C CNN
-F 2 "" H 5038 3200 50  0001 C CNN
+F 2 "Capacitor_THT:C_Disc_D5.0mm_W2.5mm_P5.00mm" H 5038 3200 50  0001 C CNN
 F 3 "~" H 5000 3350 50  0001 C CNN
 	1    5000 3350
@@
 F 0 "C6" V 4448 2700 50  0000 C CNN
 F 1 "47n" V 4539 2700 50  0000 C CNN
-F 2 "" H 4738 2550 50  0001 C CNN
+F 2 "Capacitor_THT:C_Rect_L7.2mm_W3.0mm_P5.00mm_FKS2_FKP2_MKS2_MKP2" H 4738 2550 50  0001 C CNN
 F 3 "~" H 4700 2700 50  0001 C CNN
 	1    4700 2700
@@
 F 0 "RV1" H 3581 3946 50  0000 R CNN
 F 1 "100k" H 3581 3855 50  0000 R CNN
-F 2 "" H 3650 3900 50  0001 C CNN
+F 2 "TerminalBlock:TerminalBlock_bornier-3_P5.08mm" H 3650 3900 50  0001 C CNN
 F 3 "~" H 3650 3900 50  0001 C CNN
 	1    3650 3900
@@
 F 0 "C10" V 7000 3500 50  0000 C CNN
 F 1 "470p" V 6889 3350 50  0000 C CNN
-F 2 "" H 7088 3200 50  0001 C CNN
+F 2 "Capacitor_THT:C_Disc_D5.0mm_W2.5mm_P5.00mm" H 7088 3200 50  0001 C CNN
 F 3 "~" H 7050 3350 50  0001 C CNN
 	1    7050 3350
@@
 F 0 "C9" V 6498 2700 50  0000 C CNN
 F 1 "47n" V 6589 2700 50  0000 C CNN
-F 2 "" H 6788 2550 50  0001 C CNN
+F 2 "Capacitor_THT:C_Rect_L7.2mm_W3.0mm_P5.00mm_FKS2_FKP2_MKS2_MKP2" H 6788 2550 50  0001 C CNN
 F 3 "~" H 6750 2700 50  0001 C CNN
 	1    6750 2700
@@
 F 0 "C8" V 5648 3900 50  0000 C CNN
 F 1 "100n" V 5739 3900 50  0000 C CNN
-F 2 "" H 5938 3750 50  0001 C CNN
+F 2 "Capacitor_THT:C_Rect_L7.2mm_W3.0mm_P5.00mm_FKS2_FKP2_MKS2_MKP2" H 5938 3750 50  0001 C CNN
 F 3 "~" H 5900 3900 50  0001 C CNN
 	1    5900 3900
@@
 F 0 "RV2" H 8281 3946 50  0000 R CNN
 F 1 "100k" H 8281 3855 50  0000 R CNN
-F 2 "" H 8350 3900 50  0001 C CNN
+F 2 "TerminalBlock:TerminalBlock_bornier-3_P5.08mm" H 8350 3900 50  0001 C CNN
 F 3 "~" H 8350 3900 50  0001 C CNN
 	1    8350 3900
@@
 F 0 "C11" V 7698 3600 50  0000 C CNN
 F 1 "3.9n" V 7789 3600 50  0000 C CNN
-F 2 "" H 7988 3450 50  0001 C CNN
+F 2 "Capacitor_THT:C_Rect_L7.2mm_W3.0mm_P5.00mm_FKS2_FKP2_MKS2_MKP2" H 7988 3450 50  0001 C CNN
 F 3 "~" H 7950 3600 50  0001 C CNN
 	1    7950 3600
@@
 F 0 "C13" V 8448 3900 50  0000 C CNN
 F 1 "100n" V 8539 3900 50  0000 C CNN
-F 2 "" H 8738 3750 50  0001 C CNN
+F 2 "Capacitor_THT:C_Rect_L7.2mm_W3.0mm_P5.00mm_FKS2_FKP2_MKS2_MKP2" H 8738 3750 50  0001 C CNN
 F 3 "~" H 8700 3900 50  0001 C CNN
 	1    8700 3900
@@
 F 0 "C12" H 8235 4404 50  0000 R CNN
 F 1 "10n" H 8235 4495 50  0000 R CNN
-F 2 "" H 8388 4300 50  0001 C CNN
+F 2 "Capacitor_THT:C_Rect_L7.2mm_W3.0mm_P5.00mm_FKS2_FKP2_MKS2_MKP2" H 8388 4300 50  0001 C CNN
 F 3 "~" H 8350 4450 50  0001 C CNN
 	1    8350 4450
@@
 F 0 "C14" V 9598 3600 50  0000 C CNN
 F 1 "100n" V 9689 3600 50  0000 C CNN
-F 2 "" H 9888 3450 50  0001 C CNN
+F 2 "Capacitor_THT:C_Rect_L7.2mm_W3.0mm_P5.00mm_FKS2_FKP2_MKS2_MKP2" H 9888 3450 50  0001 C CNN
 F 3 "~" H 9850 3600 50  0001 C CNN
 	1    9850 3600
@@
 L Device:CP C1
 U 1 1 60A66AE9
-P 1500 2250
-F 0 "C1" H 1618 2296 50  0000 L CNN
-F 1 "20u" H 1618 2205 50  0000 L CNN
-F 2 "" H 1538 2100 50  0001 C CNN
-F 3 "~" H 1500 2250 50  0001 C CNN
-	1    1500 2250
+P 1600 1300
+F 0 "C1" H 1718 1346 50  0000 L CNN
+F 1 "20u" H 1718 1255 50  0000 L CNN
+F 2 "Capacitor_THT:CP_Radial_D5.0mm_P2.50mm" H 1638 1150 50  0001 C CNN
+F 3 "~" H 1600 1300 50  0001 C CNN
+	1    1600 1300
 	1    0    0    -1
 $EndComp
@@
 L power:+9V #PWR01
 U 1 1 60A70E1D
-P 1500 2000
-F 0 "#PWR01" H 1500 1850 50  0001 C CNN
-F 1 "+9V" H 1515 2173 50  0000 C CNN
-F 2 "" H 1500 2000 50  0001 C CNN
-F 3 "" H 1500 2000 50  0001 C CNN
-	1    1500 2000
+P 1600 1050
+F 0 "#PWR01" H 1600 900 50  0001 C CNN
+F 1 "+9V" H 1615 1223 50  0000 C CNN
+F 2 "" H 1600 1050 50  0001 C CNN
+F 3 "" H 1600 1050 50  0001 C CNN
+	1    1600 1050
 	1    0    0    -1
 $EndComp
@@
 L power:GND #PWR02
 U 1 1 60A717C5
-P 1500 2700
-F 0 "#PWR02" H 1500 2450 50  0001 C CNN
-F 1 "GND" H 1505 2527 50  0000 C CNN
-F 2 "" H 1500 2700 50  0001 C CNN
-F 3 "" H 1500 2700 50  0001 C CNN
-	1    1500 2700
-	1    0    0    -1
-$EndComp
-Wire Wire Line
-	1500 2700 1500 2600
-Wire Wire Line
-	1500 2000 1500 2050
-Wire Wire Line
-	1050 2050 1500 2050
-Connection ~ 1500 2050
-Wire Wire Line
-	1500 2050 1500 2100
-Text Notes 750  1800 0    50   ~ 0
+P 1600 1750
+F 0 "#PWR02" H 1600 1500 50  0001 C CNN
+F 1 "GND" H 1605 1577 50  0000 C CNN
+F 2 "" H 1600 1750 50  0001 C CNN
+F 3 "" H 1600 1750 50  0001 C CNN
+	1    1600 1750
+	1    0    0    -1
+$EndComp
+Wire Wire Line
+	1600 1750 1600 1650
+Wire Wire Line
+	1600 1050 1600 1100
+Wire Wire Line
+	1150 1100 1600 1100
+Connection ~ 1600 1100
+Wire Wire Line
+	1600 1100 1600 1150
+Text Notes 850  850  0    50   ~ 0
 To DC Shroud
 Wire Wire Line
-	1050 2600 1500 2600
-Connection ~ 1500 2600
-Wire Wire Line
-	1500 2600 1500 2400
+	1150 1650 1600 1650
+Connection ~ 1600 1650
+Wire Wire Line
+	1600 1650 1600 1450
 Wire Wire Line
 	1200 3900 1300 3900
 Wire Wire Line
 	10500 3900 10400 3900
-Text Notes 800  3000 0    50   ~ 0
+Text Notes 900  2050 0    50   ~ 0
 To DC Pin
 Text Notes 6100 1550 0    50   ~ 0
@@
 Text GLabel 1200 3900 0    50   Input ~ 0
 in
-Text GLabel 1050 2050 0    50   Input ~ 0
+Text GLabel 1150 1100 0    50   Input ~ 0
 pwr
-Text GLabel 1050 2600 0    50   Input ~ 0
+Text GLabel 1150 1650 0    50   Input ~ 0
 gnd
 $Comp
@@
 Wire Wire Line
 	3900 6500 4100 6500
+$Comp
+L Device:D D5
+U 1 1 6092CF40
+P 2150 1300
+F 0 "D5" V 2104 1379 50  0000 L CNN
+F 1 "1n4001" V 2195 1379 50  0000 L CNN
+F 2 "Diode_THT:D_DO-41_SOD81_P10.16mm_Horizontal" H 2150 1300 50  0001 C CNN
+F 3 "~" H 2150 1300 50  0001 C CNN
+	1    2150 1300
+	0    1    1    0
+$EndComp
+Wire Wire Line
+	2150 1150 2150 1100
+Wire Wire Line
+	2150 1100 1600 1100
+Wire Wire Line
+	2150 1450 2150 1650
+Wire Wire Line
+	2150 1650 1600 1650
 $EndSCHEMATC
