File: staypuft.kicad_pcb (KiCad board)
At the start: 2 copper layers, 53 parts, among them J1 Conn_01x04_Male, Q1 2N5088, Q2 2N5088, Q3 2N5088, Q4 2N5088

Commit message: grouping on pcb in prog
Parts:
- moved D2 248.8 mm to (261.0, 85.0), turned to 270 degrees
- moved R9 222.6 mm to (242.0, 82.0)
- moved R2 218.1 mm to (238.0, 107.0), turned to 180 degrees
- moved R11 212.6 mm to (242.0, 77.0)
- moved Q2 208.1 mm to (257.0, 76.0), turned to 270 degrees
- moved TP4 202.9 mm to (266.0, 85.0), turned to 270 degrees
- moved C6 196.7 mm to (270.0, 81.0), turned to 90 degrees
- moved D1 195.2 mm to (257.0, 95.0), turned to 90 degrees
- moved R13 193.0 mm to (228.0, 87.0)
- moved R10 192.6 mm to (252.0, 92.0), turned to 180 degrees
- moved C7 191.4 mm to (264.0, 81.0), turned to 90 degrees
- moved C8 183.1 mm to (250.0, 155.0)
- moved R12 178.5 mm to (238.0, 77.0), turned to 180 degrees
- moved R8 177.8 mm to (242.0, 87.0)
- moved C12 174.5 mm to (228.0, 162.0)
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Routing:
- net Net-(C7-Pad1): track 0.00 -> 48.5 mm
- net Net-(C10-Pad1): track 0.00 -> 48.3 mm
- net Net-(C2-Pad1): track 0.00 -> 32.5 mm
- net Net-(C10-Pad2): track 0.00 -> 31.7 mm
- net Net-(C6-Pad2): track 0.00 -> 26.0 mm
- net Net-(C14-Pad2): track 0.00 -> 24.6 mm
- net Net-(C3-Pad1): track 0.00 -> 24.1 mm
- net Net-(C6-Pad1): track 0.00 -> 20.7 mm
- net Net-(C13-Pad1): track 0.00 -> 18.8 mm
- net Net-(C9-Pad1): track 0.00 -> 15.7 mm
- net Net-(Q4-Pad1): track 0.00 -> 11.1 mm
- net gnd: track 0.00 -> 10.0 mm
- net Net-(Q3-Pad1): track 0.00 -> 9.41 mm
- net Net-(Q2-Pad1): track 0.00 -> 9.25 mm
- net Net-(Q1-Pad1): track 0.00 -> 4.84 mm
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Other:
- board text added: "Do I need to flip these pins for the pots? check the blender."

Commit message: still working on pcb
Parts:
- moved TP4 113.8 mm to (152.5, 76.5), turned to 0 degrees
- moved R12 111.8 mm to (137.0, 125.0), turned to 90 degrees
- moved R14 111.0 mm to (132.0, 115.0), turned to 270 degrees
- moved R7 110.3 mm to (171.5, 74.5), turned to 270 degrees
- moved Q2 109.7 mm to (147.5, 83.0), turned to 0 degrees
- moved TP5 109.6 mm to (147.5, 76.5), turned to 90 degrees
- moved C5 109.1 mm to (177.0, 80.0), turned to 90 degrees
- moved R16 108.5 mm to (122.0, 115.0), turned to 270 degrees
- moved R13 104.8 mm to (127.0, 115.0), turned to 270 degrees
- moved C6 103.7 mm to (166.5, 74.5), turned to 270 degrees
- moved TP6 101.3 mm to (122.5, 110.0), turned to 0 degrees
- moved D1 99.6 mm to (158.0, 84.0)
- moved D2 99.6 mm to (162.0, 74.0)
- moved Q3 98.0 mm to (126.5, 110.0), turned to 0 degrees
- moved R15 96.2 mm to (142.0, 115.0), turned to 270 degrees
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Routing:
- net Net-(C13-Pad2): track 0.00 -> 17.1 mm
- net Net-(C12-Pad2): track 0.00 -> 15.9 mm
- net Net-(C6-Pad2): track 26.0 -> 40.0 mm
- net Net-(C5-Pad1): track 0.00 -> 11.8 mm
- net Net-(C6-Pad1): track 20.7 -> 9.27 mm
- net Net-(C7-Pad1): track 48.5 -> 37.7 mm
- net gnd: track 10.0 -> 0.00 mm
- net Net-(C13-Pad1): track 18.8 -> 26.5 mm
- net Net-(C5-Pad2): track 0.00 -> 6.00 mm
- net Net-(R6-Pad2): track 0.00 -> 5.87 mm
- net Net-(Q4-Pad1): track 11.1 -> 5.55 mm
- net Net-(C14-Pad2): track 24.6 -> 19.2 mm
- net Net-(C14-Pad1): track 0.00 -> 5.00 mm
- net Net-(C10-Pad2): track 31.7 -> 36.3 mm
- net Net-(C11-Pad1): track 0.00 -> 4.50 mm
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Other:
- board outline added: 68 x 77.5 mm
- board text removed: "Do I need to flip these pins for the pots? check the blender."

Commit message: rough pcb done, align todo
Parts:
- moved R18 93.9 mm to (141.0, 73.0)
- moved C11 87.4 mm to (146.5, 76.5), turned to 270 degrees
- moved C8 72.2 mm to (136.5, 94.0), turned to 90 degrees
- moved C12 71.6 mm to (157.0, 81.5)
- moved R17 67.4 mm to (162.5, 75.5)
- moved C7 43.5 mm to (158.0, 89.5), turned to 0 degrees
- moved Q4 38.1 mm to (128.5, 118.0), turned to 90 degrees
- moved R20 36.0 mm to (159.5, 112.5), turned to 180 degrees
- moved C1 34.7 mm to (162.0, 121.5), turned to 90 degrees
- moved C4 34.3 mm to (167.5, 76.0), turned to 270 degrees
- moved TP7 33.0 mm to (133.0, 113.5)
- moved R22 32.2 mm to (146.5, 117.5), turned to 180 degrees
- moved C6 30.5 mm to (149.0, 99.5), turned to 0 degrees
- moved D5 30.1 mm to (167.0, 121.5), turned to 0 degrees
- moved TP5 30.0 mm to (162.5, 102.5)
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Routing:
- net pwr: track 4.37 -> 111.8 mm
- net out: track 0.00 -> 85.0 mm
- net Net-(C13-Pad1): track 26.5 -> 73.1 mm
- net Net-(C14-Pad2): track 19.2 -> 51.9 mm
- net Net-(C10-Pad2): track 36.3 -> 53.9 mm
- net in: track 0.27 -> 17.7 mm
- net Net-(C8-Pad1): track 0.00 -> 15.9 mm
- net Net-(C10-Pad1): track 45.5 -> 58.7 mm
- net Net-(C6-Pad2): track 40.0 -> 51.4 mm
- net Net-(C11-Pad1): track 4.50 -> 14.2 mm
- net Net-(C13-Pad2): track 17.1 -> 7.50 mm
- net Net-(C4-Pad1): track 0.00 -> 8.83 mm
- net Net-(C3-Pad1): track 22.6 -> 31.3 mm
- net Net-(C9-Pad1): track 18.4 -> 11.4 mm
- net Net-(C2-Pad1): track 30.4 -> 23.8 mm
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Other:
- board size 68 x 77.5 mm -> 68 x 59 mm

Commit message: final touches done on pcb
Parts:
- added G***: LOGO, eric:nayong, B.Cu at (155.0, 112.8)
- added REF**: MountingHole_2.2mm_M2_DIN965, MountingHole:MountingHole_2.2mm_M2_DIN965, F.Cu at (121.2, 121.2)
- moved C4 0.36 mm to (167.5, 75.6)
- moved C5 0.36 mm to (177.0, 80.6)
- moved R22 0.35 mm to (146.8, 117.8)
- moved D1 0.16 mm to (155.2, 94.7)
- moved D4 0.16 mm to (126.8, 80.5)
- moved D5 0.16 mm to (166.8, 121.5)
- moved R12 0.16 mm to (146.7, 104.0)
- moved R19 0.16 mm to (149.3, 108.5)
- moved R7 0.16 mm to (172.0, 75.3)
- moved R2 0.09 mm to (181.6, 114.0)
- renumbered TP5 to FB1, TP6 to FB1, TP4 to FB2, TP7 to FB2, RV1 to Sustain, RV2 to Tone
Routing:
- net Net-(C10-Pad1): track 58.7 -> 59.7 mm
- added copper zone on B.Cu, net gnd
Other:
- board text added: ""enjoy responsibly""
- board text added: "-"
- board text added: "->"
- board text added: "9v"
- board text added: "Another Idiot Project"
- board text added: "IN"
- board text added: "OUT"
- board text added: "Volume"
- board text added: "staypuft fuzz"
